File: STMPod/STMPod/STMPod.sch (KiCad schematic (older format))
At the start: 6 parts, among them J1 Conn_01x04_Male, SW1 SW_SPST, U1 STM32F030F4Px, Y1 Resonator

Commit message: Schematic done, Placement Done
Schematic done and placement for PCB, as well as initial routing. Need to finish power planes
Parts:
- added C1, C2: 1.0uF, Capacitor_SMD:C_0603_1608Metric, symbol Device:C
- added C3, C4: 0.1uF, Capacitor_SMD:C_0603_1608Metric, symbol Device:C
- added D1, D2: LED AMBER 2.9V 5mA, LED_SMD:LED_0603_1608Metric, symbol Device:LED
- added J2, J3: Conn_01x12_Male, Connector_PinHeader_2.54mm:PinHeader_1x12_P2.54mm_Vertical, symbol Connector:Conn_01x12_Male
- added J4: USB_B_Mini, Connector_USB:USB_Mini-B_Lumberg_2486_01_Horizontal, symbol Connector:USB_B_Mini
- added R3, R4: 220, Resistor_SMD:R_0603_1608Metric, symbol Device:R_US
- added U2: MIC2920A-3.3WS, Package_TO_SOT_SMD:SOT-223, symbol AK_Power:MIC2920A-3.3WS
- gave numbers to parts that had none: 1
Connections:
- net labels added: +5V, GND, PA0, PA1, PA10, PA2, PA3, PA4, PA5, PA6, PA7, PA9, PB1
- wire segments 40 -> 105
- no-connect marks 0 -> 3
Other:
- note added: "CAN BE NP IF DESIRED\n"
- note added: "CAP ON EACH VDD PIN (VDD, VDDA)\n"

Commit message: PCB Finished
Done with layout, 3D preview, next step is generating gerbers
Connections:
- net labels removed: GND
- wire segments 105 -> 106
Changed lines of the file:
@@
 EESchema Schematic File Version 4
+LIBS:STMPod-cache
 EELAYER 26 0
 EELAYER END
@@
 Wire Wire Line
 	6850 2300 6400 2300
-Wire Wire Line
-	6850 2200 6400 2200
 Wire Wire Line
 	6850 2000 6400 2000
@@
 Text Label 6550 2300 0    50   ~ 0
 PB1
-Text Label 6550 2200 0    50   ~ 0
-GND
 $Comp
 L power:+3.3V #PWR0122
@@
 Wire Wire Line
 	6250 2100 6250 2050
+$Comp
+L power:GNDREF #PWR?
+U 1 1 5B5AAF2E
+P 6250 2300
+F 0 "#PWR?" H 6250 2050 50  0001 C CNN
+F 1 "GNDREF" H 6050 2250 50  0000 C CNN
+F 2 "" H 6250 2300 50  0001 C CNN
+F 3 "" H 6250 2300 50  0001 C CNN
+	1    6250 2300
+	1    0    0    -1
+$EndComp
+Wire Wire Line
+	6250 2200 6250 2300
+Wire Wire Line
+	6250 2200 6850 2200
 $EndSCHEMATC
