File: STMPod/STMPod/_autosave-STMPod.kicad_pcb (KiCad board)
At the start: 2 copper layers, 19.6 x 32.3 mm, 19 parts, among them J1 Conn_01x04_Male, J2 Conn_01x12_Male, J3 Conn_01x12_Male, J4 USB_B_Mini, SW1 SW_SPST, U1 STM32F030F4Px, U2 MIC2920A-3.3WS, Y1 Resonator

Commit message: STMPod & MotorPod Mini
Prepped STMPod for manufacture,
MotorPodMini designed in one sitting (I'm so bored...)
Parts:
- U2: value MIC2920A-3.3WS -> AZ1117-3.3; footprint Package_TO_SOT_SMD:SOT-223 -> Package_TO_SOT_SMD:SOT-223-3_TabPin2
- moved C2 3.14 mm to (172.1, 84.8), turned to 270 degrees
- moved U2 3.06 mm to (177.3, 82.9), turned to 0 degrees
Connections:
- U2 pad 1: +5V -> GNDREF
- U2 pad 2: GNDREF -> +3V3
- U2 pad 3: +3V3 -> +5V
Routing:
- net +3V3: track 66.7 -> 73.1 mm
- net GNDREF: track 47.1 -> 49.3 mm
- net +5V: track 20.9 -> 22.0 mm
