File: EFMPod/EFMPod/_saved_EFMPod.sch (KiCad schematic (older format))
At the start: 49 parts, among them J1 Conn_01x04, J2 UJ2-MBH-1-SMT-TR, J3 Conn_02x18_Odd_Even, SW1 SW_Push, SW2 SW_Push, SW3 SW_Push, U1 AZ1117CH-3_3TRG1, U2 EFM32HG322F64, Y2 Crystal_GND3

Commit message: PCB Placement done, routing started
Placement done, signal routing mostly done, board outline generated, mounting holes placed
Parts:
- gave numbers to parts that had none: 1
Other:
- note added: "102-4003-1-ND"
