File: EFMPod/EFMPod/EFMPod.sch (KiCad schematic (older format))
At the start: 49 parts, among them J1 Conn_01x04, J2 UJ2-MBH-1-SMT-TR, J3 Conn_02x18_Odd_Even, SW1 SW_Push, SW2 SW_Push, SW3 SW_Push, U1 AZ1117CH-3_3TRG1, U2 EFM32HG322F64, Y2 Crystal_GND3

Commit message: Placement Progress`
Added ARM debug header, some more routing & placement, added correct switches
Parts:
- removed J1: Conn_01x04, Connector_PinHeader_2.54mm:PinHeader_1x04_P2.54mm_Vertical, symbol Connector_Generic:Conn_01x04
- added J1: Conn_02x05_Odd_Even, Connector_PinHeader_1.27mm:PinHeader_2x05_P1.27mm_Vertical_SMD, symbol Connector_Generic:Conn_02x05_Odd_Even
- gave numbers to parts that had none: 1
Connections:
- wire segments 239 -> 244
- no-connect marks 0 -> 3
Other:
- note added: "102-4003-1-ND"

Commit message: Layout done
Layout done, silk & gerbers next
Parts:
- removed Y1: 24MHz, Crystal:Crystal_HC49-U_Vertical, symbol Device:Crystal
- added Y1: Crystal_GND24, Crystal:Crystal_SMD_SeikoEpson_FA238-4Pin_3.2x2.5mm_HandSoldering, symbol Device:Crystal_GND24
Connections:
- wire segments 244 -> 250
Changed lines of the file:
@@
 $EndComp
 Wire Wire Line
-	6050 7550 6600 7550
-$Comp
-L Device:Crystal Y1
-U 1 1 5B8D9059
-P 6300 6900
-F 0 "Y1" H 6300 7168 50  0000 C CNN
-F 1 "24MHz" H 6300 7077 50  0000 C CNN
-F 2 "Crystal:Crystal_HC49-U_Vertical" H 6300 6900 50  0001 C CNN
-F 3 "~" H 6300 6900 50  0001 C CNN
-	1    6300 6900
-	1    0    0    -1
-$EndComp
+	6050 7550 6300 7550
 Wire Wire Line
 	6050 6900 6150 6900
@@
 	2100 4150 2100 3950
 NoConn ~ 2700 3950
+$Comp
+L Device:Crystal_GND24 Y1
+U 1 1 5B92BA1F
+P 6300 6900
+F 0 "Y1" H 6450 7150 50  0000 L CNN
+F 1 "Crystal_GND24" H 6450 7050 50  0000 L CNN
+F 2 "Crystal:Crystal_SMD_SeikoEpson_FA238-4Pin_3.2x2.5mm_HandSoldering" H 6300 6900 50  0001 C CNN
+F 3 "~" H 6300 6900 50  0001 C CNN
+	1    6300 6900
+	1    0    0    -1
+$EndComp
+Wire Wire Line
+	6300 7100 6300 7550
+Connection ~ 6300 7550
+Wire Wire Line
+	6300 7550 6600 7550
+Wire Wire Line
+	6300 6700 6300 6650
+Wire Wire Line
+	6300 6650 5700 6650
+Wire Wire Line
+	5700 6650 5700 7550
+Wire Wire Line
+	5700 7550 6050 7550
+Connection ~ 6050 7550
 $EndSCHEMATC
