File: DebugAdapter/DebugAdapter/DebugAdapter.sch (KiCad schematic (older format))
At the start: 6 parts

Commit message: Closed KiCAD, updated files
Parts:
- gave numbers to parts that had none: 6
Changed lines of the file:
@@
 $EndDescr
 $Comp
-L Connector_Generic:Conn_02x05_Odd_Even J?
+L Connector_Generic:Conn_02x05_Odd_Even J1
 U 1 1 5C7DECA4
 P 5000 3400
-F 0 "J?" H 5050 3817 50  0000 C CNN
+F 0 "J1" H 5050 3817 50  0000 C CNN
 F 1 "Conn_02x05_Odd_Even" H 5050 3726 50  0000 C CNN
 F 2 "Connector_PinHeader_1.27mm:PinHeader_2x05_P1.27mm_Vertical_SMD" H 5000 3400 50  0001 C CNN
@@
 $EndComp
 $Comp
-L Connector_Generic:Conn_01x04 J?
+L Connector_Generic:Conn_01x04 J2
 U 1 1 5C7DEDA9
 P 6650 3300
-F 0 "J?" H 6730 3292 50  0000 L CNN
+F 0 "J2" H 6730 3292 50  0000 L CNN
 F 1 "Conn_01x04" H 6730 3201 50  0000 L CNN
 F 2 "Connector_PinHeader_2.54mm:PinHeader_1x04_P2.54mm_Horizontal" H 6650 3300 50  0001 C CNN
@@
 $EndComp
 $Comp
-L power:GND #PWR?
+L power:GND #PWR0101
 U 1 1 5C7DEE80
 P 6350 3600
-F 0 "#PWR?" H 6350 3350 50  0001 C CNN
+F 0 "#PWR0101" H 6350 3350 50  0001 C CNN
 F 1 "GND" H 6355 3427 50  0000 C CNN
 F 2 "" H 6350 3600 50  0001 C CNN
@@
 SWCLK
 $Comp
-L power:+3.3V #PWR?
+L power:+3.3V #PWR0102
 U 1 1 5C7DEF0C
 P 6350 3100
-F 0 "#PWR?" H 6350 2950 50  0001 C CNN
+F 0 "#PWR0102" H 6350 2950 50  0001 C CNN
 F 1 "+3.3V" H 6365 3273 50  0000 C CNN
 F 2 "" H 6350 3100 50  0001 C CNN
@@
 NoConn ~ 5300 3600
 $Comp
-L power:+3.3V #PWR?
+L power:+3.3V #PWR0103
 U 1 1 5C7DF29F
 P 4550 3100
-F 0 "#PWR?" H 4550 2950 50  0001 C CNN
+F 0 "#PWR0103" H 4550 2950 50  0001 C CNN
 F 1 "+3.3V" H 4565 3273 50  0000 C CNN
 F 2 "" H 4550 3100 50  0001 C CNN
@@
 	4550 3200 4800 3200
 $Comp
-L power:GND #PWR?
+L power:GND #PWR0104
 U 1 1 5C7DF33A
 P 4550 3650
-F 0 "#PWR?" H 4550 3400 50  0001 C CNN
+F 0 "#PWR0104" H 4550 3400 50  0001 C CNN
 F 1 "GND" H 4555 3477 50  0000 C CNN
 F 2 "" H 4550 3650 50  0001 C CNN
@@
 NoConn ~ 4800 3600
 $Comp
-L Device:Battery BT?
+L Device:Battery BT1
 U 1 1 5C7DFB6B
 P 1600 3350
-F 0 "BT?" H 1708 3396 50  0000 L CNN
+F 0 "BT1" H 1708 3396 50  0000 L CNN
 F 1 "Battery" H 1708 3305 50  0000 L CNN
 F 2 "Battery:BatteryHolder_Keystone_2468_2xAAA" V 1600 3410 50  0001 C CNN
@@
 $EndComp
 $Comp
-L power:GND #PWR?
+L power:GND #PWR0105
 U 1 1 5C7DFD25
 P 1600 3650
-F 0 "#PWR?" H 1600 3400 50  0001 C CNN
+F 0 "#PWR0105" H 1600 3400 50  0001 C CNN
 F 1 "GND" H 1605 3477 50  0000 C CNN
 F 2 "" H 1600 3650 50  0001 C CNN
@@
 	1600 3550 1600 3650
 $Comp
-L power:+BATT #PWR?
+L power:+BATT #PWR0106
 U 1 1 5C7DFFE6
 P 1600 3100
-F 0 "#PWR?" H 1600 2950 50  0001 C CNN
+F 0 "#PWR0106" H 1600 2950 50  0001 C CNN
 F 1 "+BATT" H 1615 3273 50  0000 C CNN
 F 2 "" H 1600 3100 50  0001 C CNN
@@
 $EndComp
 $Comp
-L Switch:SW_SPDT SW?
+L Switch:SW_SPDT SW1
 U 1 1 5C7E06A2
 P 2950 3350
-F 0 "SW?" H 2950 3635 50  0000 C CNN
+F 0 "SW1" H 2950 3635 50  0000 C CNN
 F 1 "SW_SPDT" H 2950 3544 50  0000 C CNN
 F 2 "Button_Switch_SMD:SW_SPDT_CK-JS102011SAQN" H 2950 3350 50  0001 C CNN
@@
 $EndComp
 $Comp
-L power:+BATT #PWR?
+L power:+BATT #PWR0107
 U 1 1 5C7E0B94
 P 2600 3100
-F 0 "#PWR?" H 2600 2950 50  0001 C CNN
+F 0 "#PWR0107" H 2600 2950 50  0001 C CNN
 F 1 "+BATT" H 2615 3273 50  0000 C CNN
 F 2 "" H 2600 3100 50  0001 C CNN
@@
 	2600 3350 2750 3350
 $Comp
-L power:+3.3V #PWR?
+L power:+3.3V #PWR0108
 U 1 1 5C7E0D87
 P 3650 3100
-F 0 "#PWR?" H 3650 2950 50  0001 C CNN
+F 0 "#PWR0108" H 3650 2950 50  0001 C CNN
 F 1 "+3.3V" H 3665 3273 50  0000 C CNN
 F 2 "" H 3650 3100 50  0001 C CNN
@@
 NoConn ~ 3150 3450
 $Comp
-L Device:R_US R?
+L Device:R_US R1
 U 1 1 5C7E2075
 P 3650 3850
-F 0 "R?" H 3718 3896 50  0000 L CNN
+F 0 "R1" H 3718 3896 50  0000 L CNN
 F 1 "1.4k" H 3718 3805 50  0000 L CNN
 F 2 "Resistor_SMD:R_0603_1608Metric_Pad1.05x0.95mm_HandSolder" V 3690 3840 50  0001 C CNN
@@
 $EndComp
 $Comp
-L Device:LED D?
+L Device:LED D1
 U 1 1 5C7E20FB
 P 3650 3450
-F 0 "D?" V 3688 3333 50  0000 R CNN
+F 0 "D1" V 3688 3333 50  0000 R CNN
 F 1 "LED" V 3597 3333 50  0000 R CNN
 F 2 "Diode_SMD:D_0603_1608Metric_Pad1.05x0.95mm_HandSolder" H 3650 3450 50  0001 C CNN
@@
 	3650 3600 3650 3700
 $Comp
-L power:GND #PWR?
+L power:GND #PWR0109
 U 1 1 5C7E2D9D
 P 3650 4000
-F 0 "#PWR?" H 3650 3750 50  0001 C CNN
+F 0 "#PWR0109" H 3650 3750 50  0001 C CNN
 F 1 "GND" H 3655 3827 50  0000 C CNN
 F 2 "" H 3650 4000 50  0001 C CNN
